File: Design Files/D-DAQ Mainboard.brd (EAGLE design)
At the start: 99.8 x 49.9 mm, 123 parts, among them Y1 16.368 MHz, Y2 DS1099

Commit message: Update to Proto v3.6. Please visit the following for details: http://hackaday.io/project/964/log/4782
Parts:
- removed R13: 10k, resistor:R0603
- removed U$2, U$3, U$4, U$5: (no value), holes:2,8
- added C10, C11, C9: 4.7uF, Parts for D-DAQ:SMD-0603
- 10&11, 12&13, 4&5, 8&9, IMP.: device Parts for DC MF Gauge:USB-MICRO-B-VERT -> Parts for D-DAQ:USB-MICRO-B-VERT
- 14V-REG: device Parts for DC MF Gauge:SOT-223-6 -> Parts for D-DAQ:SOT-223-6
- 2.8V: device Parts for DC MF Gauge:SOT-23-5 -> Parts for D-DAQ:SOT-23-5
- 3.3V-TOGGLE-1, 3.3V-TOGGLE-2, 3.3V-TOGGLE-5: device Parts for DC MF Gauge:SOP-4--CPC1017N -> Parts for D-DAQ:SOP-4--CPC1017N
- 5V-REG: device Parts for DC MF Gauge:SOT-223-5 -> Parts for D-DAQ:SOT-223-5
- 5V-TOGGLE-1, 5V-TOGGLE-2, 5V-TOGGLE-5: device Parts for DC MF Gauge:SOP-4--CPC1117N -> Parts for D-DAQ:SOP-4--CPC1117N
- 6&7+: device Parts for DC MF Gauge:USB-MICRO-AB-FLAT -> Parts for D-DAQ:USB-MICRO-AB-FLAT
- AS7C31026B: device Parts for DC MF Gauge:TSOP-44 -> Parts for D-DAQ:TSOP-44
- AUX-PRESS: device con-molex-alt:PC-1771101 -> Parts for D-DAQ:PC-1771101
- C1, C117, C118, C119, C121, C122, C123, C124, C125, C126, C127, C2, C4, C5, C6, C7, C8: device resistor:C0603K -> Parts for D-DAQ:SMD-0603
- C1.1, C1.2: device resistor:C1206 -> Parts for D-DAQ:SMD-1812-EDGE
- C2.1, C2.2, C21, C22, C3, C31: device resistor:C1206 -> Parts for D-DAQ:SMD-1206
- CAN-BUS, DATA: device Parts for DC MF Gauge:USB-MINI-B-VERT -> Parts for D-DAQ:USB-MINI-B-VERT
- D1, D2, D3: device Parts for D-DAQ:SOD-123W -> Parts for D-DAQ:DO-219AB-2
- DISP-1, DISP-2, DISP-3: value DP3AR020SU32JQ1-STANDARD -> (none); device con-molex-alt:DP3AR020SU32JQ1-STANDARD -> Parts for D-DAQ:JAE-MDP-STD
- EGT, POWER: device Parts for DC MF Gauge:PC-1702610 -> Parts for D-DAQ:PC-1702610
- EGT-AMP: device Parts for DC MF Gauge:SOT-8 -> Parts for D-DAQ:SOT-8
- F0, F1, F10, F11, F12, F13, F14, F2, F3, F4, F5, F6, F7, F8, F9, R1, R10, R11, R12, R127, R129, R130, R131, R132, R133, R135, R136, R138, R139, R14, R140, R141, R142, R145, R146, R147, R15, R2, R20, R21, R3, R31, R32, R4, R5, R6, R7, R8, R9: device resistor:R0603 -> Parts for D-DAQ:SMD-0603
- JTAG: value (none) -> HEADER-X4; device pinhead:1X04 -> Parts for D-DAQ:HEADER-X4
- L1: device Parts for DC MF Gauge:7443551XXX -> Parts for D-DAQ:7443551XXX
- LATCH-HIGH, LATCH-LOW: device Parts for DC MF Gauge:TSSOP-20 -> Parts for D-DAQ:TSSOP-20
- MAIN-SMPS: device Parts for DC MF Gauge:QFN-14 -> Parts for D-DAQ:QFN-14
- MICRO-SD: device Parts for DC MF Gauge:SCHA4B0400 -> Parts for D-DAQ:SCHA4B0400
- MMA8652FC: device Parts for DC MF Gauge:QFN-12 -> Parts for D-DAQ:QFN-12
- MPL3115A101: device Parts for DC MF Gauge:LGA-8 -> Parts for D-DAQ:LGA-8
- NBPLANN100PAUNV: device Parts for DC MF Gauge:LEADLESS-SMT -> Parts for D-DAQ:LEADLESS-SMT
- PIC32MX: device Parts for DC MF Gauge:TQFP-100 -> Parts for D-DAQ:TQFP-100-12X12
- SC18IS602B: device Parts for DC MF Gauge:TSSOP-16 -> Parts for D-DAQ:TSSOP-16
- U$6, U$7: device SparkFun:OSHW-LOGO-S -> Parts for D-DAQ:OSHW-LOGO-S
- Y1: value 16.368 MHz -> XTC7009; device Parts for DC MF Gauge:XTC7009 -> Parts for D-DAQ:3.2X2.5MM
- Y2: device Parts for DC MF Gauge:SOIC-8 -> Parts for D-DAQ:SOIC-8
- moved R136 3.20 mm to (94.5, 23.5), flipped to the bottom, turned to 90 degrees
- moved R132 1.49 mm to (96.7, 19.3), turned to 180 degrees
- moved L1 1.43 mm to (15.6, 6.48)
- moved C6 0.98 mm to (19.9, 23.8), turned to 0 degrees
- moved C1.2 0.76 mm to (16.1, 15.0)
- moved C3 0.57 mm to (23.3, 13.5)
- moved C21 0.27 mm to (13.8, 42.4)
- moved C1.1 0.19 mm to (16.1, 26.6)
- turned D3 to 270 degrees
- turned D1 to 180 degrees
- turned D2 to 90 degrees
Connections:
- removed net OE0: R13.1, Y2.5
- new net BOOST-SSR: 3.3V-TOGGLE-2.1, 5V-TOGGLE-2.2, C11.2
- new net USB-SSR: 3.3V-TOGGLE-1.1, 5V-TOGGLE-1.2, C10.2
- net 100-PSI-SENSOR-RES: no longer 3.3V-TOGGLE-2.1
- net 12V-INPUT: now also D2.P$1; no longer D2.P$2
- net 14V-INPUT: now also D3.P$2; no longer D3.P$1
- net 3.3V-RAIL: now also 3.3V-TOGGLE-1.3, 3.3V-TOGGLE-2.3; no longer 3.3V-TOGGLE-1.4, 3.3V-TOGGLE-2.4
- net 5V-RAIL: now also 5V-TOGGLE-1.4, Y2.5; no longer 5V-TOGGLE-1.3
- net AUTO-DETECT: no longer 3.3V-TOGGLE-1.1
- net BOOST-PWR: now also 3.3V-TOGGLE-2.4; no longer 3.3V-TOGGLE-2.3
- net CP-PUMP: now also D2.P$2, D3.P$1; no longer D2.P$1, D3.P$2
- net EGT-NEG-IN: now also R136.1; no longer R136.2
- net EGT-SHTDWN: now also R132.2; no longer R132.1
- net GND: now also C10.1, C11.1, C9.2, D1.P$1, R132.1, R136.2; no longer 5V-TOGGLE-1.2, 5V-TOGGLE-2.2, D1.P$2, R13.2, R132.2, R136.1
- net ICSP-SSR: now also C9.1
- net PWR-GND: now also D1.P$2; no longer D1.P$1
- net USB-PWR: now also 3.3V-TOGGLE-1.4, 5V-TOGGLE-1.3; no longer 3.3V-TOGGLE-1.3, 5V-TOGGLE-1.4
Routing:
- net 3.3V-RAIL: track 361.8 -> 379.3 mm, vias 33 -> 36
- net GND: track 27.8 -> 19.2 mm
- net BOOST-SSR: track 0.00 -> 6.47 mm
- net USB-SSR: track 0.00 -> 5.54 mm
- net AUTO-DETECT: track 16.9 -> 11.4 mm, vias 4 -> 2
- net USB-PWR: track 50.5 -> 47.3 mm, vias 3 -> 2
- net 5V-RAIL: track 169.3 -> 172.4 mm, vias 16 -> 13
- net EGT-NEG-IN: track 28.6 -> 25.9 mm, vias 5 -> 4
- net OE0: track 2.46 -> 0.00 mm
- net 12V-INPUT: track 73.4 -> 71.4 mm, vias 17 -> 16
- net EGT-POS-IN: track 19.2 -> 21.1 mm
- net BOOST-PWR: track 19.1 -> 17.4 mm, vias 2 -> 1
- net 100-PSI-SENSOR-RES: track 11.6 -> 10.0 mm, vias 2 -> 0
- net 12V-SS: track 3.83 -> 2.63 mm
- net ICSP-SSR: track 2.09 -> 2.96 mm
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Other:
- outline, holes or cut-outs redrawn
- board text added: "D-DAQ Proto 3.6"
- board text removed: "D-DAQ Proto 3.5"

Commit message: v3.6.1 No major changes, just cleanup and moving to Eagle v6.6 files
Parts:
- 3.3V-TOGGLE-1, 3.3V-TOGGLE-2, 3.3V-TOGGLE-5: device Parts for D-DAQ:SOP-4--CPC1017N -> Parts for D-DAQ:SOP-4-NO
- 5V-REG: device Parts for D-DAQ:SOT-223-5 -> Parts for D-DAQ:SOT-223-4
- 5V-TOGGLE-1, 5V-TOGGLE-2, 5V-TOGGLE-5: device Parts for D-DAQ:SOP-4--CPC1117N -> Parts for D-DAQ:SOP-4-NC
Changed lines of the file:
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@@
 <?xml version="1.0" encoding="utf-8"?>
 <!DOCTYPE eagle SYSTEM "eagle.dtd">
-<eagle version="6.4">
+<eagle version="6.6.0">
 <drawing>
 <settings>
@@
 <layer number="51" name="tDocu" color="7" fill="1" visible="yes" active="yes"/>
 <layer number="52" name="bDocu" color="7" fill="1" visible="yes" active="yes"/>
-<layer number="53" name="tGND_GNDA" color="7" fill="9" visible="no" active="no"/>
-<layer number="54" name="bGND_GNDA" color="1" fill="9" visible="no" active="no"/>
-<layer number="56" name="wert" color="7" fill="1" visible="no" active="no"/>
 <layer number="91" name="Nets" color="2" fill="1" visible="no" active="no"/>
 <layer number="92" name="Busses" color="1" fill="1" visible="no" active="no"/>
@@
 <layer number="97" name="Info" color="7" fill="1" visible="no" active="no"/>
 <layer number="98" name="Guide" color="6" fill="1" visible="no" active="no"/>
-<layer number="99" name="SpiceOrder" color="5" fill="1" visible="no" active="no"/>
-<layer number="100" name="Muster" color="7" fill="1" visible="no" active="no"/>
-<layer number="101" name="Patch_Top" color="12" fill="4" visible="no" active="yes"/>
-<layer number="102" name="Vscore" color="7" fill="1" visible="no" active="yes"/>
-<layer number="103" name="tMap" color="7" fill="1" visible="no" active="yes"/>
-<layer number="104" name="Name" color="16" fill="1" visible="no" active="yes"/>
-<layer number="105" name="tPlate" color="7" fill="1" visible="no" active="yes"/>
-<layer number="106" name="bPlate" color="7" fill="1" visible="no" active="yes"/>
-<layer number="107" name="Crop" color="7" fill="1" visible="no" active="yes"/>
-<layer number="116" name="Patch_BOT" color="9" fill="4" visible="no" active="yes"/>
-<layer number="121" name="_tsilk" color="7" fill="1" visible="no" active="yes"/>
-<layer number="122" name="_bsilk" color="7" fill="1" visible="no" active="yes"/>
-<layer number="125" name="_tNames" color="7" fill="1" visible="no" active="yes"/>
-<layer number="144" name="Drill_legend" color="7" fill="1" visible="no" active="yes"/>
-<layer number="151" name="HeatSink" color="7" fill="1" visible="no" active="yes"/>
-<layer number="200" name="200bmp" color="1" fill="10" visible="no" active="yes"/>
-<layer number="201" name="201bmp" color="2" fill="10" visible="no" active="yes"/>
-<layer number="202" name="202bmp" color="3" fill="10" visible="no" active="yes"/>
-<layer number="203" name="203bmp" color="4" fill="10" visible="no" active="yes"/>
-<layer number="204" name="204bmp" color="5" fill="10" visible="no" active="yes"/>
-<layer number="205" name="205bmp" color="6" fill="10" visible="no" active="yes"/>
-<layer number="206" name="206bmp" color="7" fill="10" visible="no" active="yes"/>
-<layer number="207" name="207bmp" color="8" fill="10" visible="no" active="yes"/>
-<layer number="208" name="208bmp" color="9" fill="10" visible="no" active="yes"/>
-<layer number="209" name="209bmp" color="7" fill="1" visible="no" active="yes"/>
-<layer number="210" name="210bmp" color="7" fill="1" visible="no" active="yes"/>
-<layer number="211" name="211bmp" color="7" fill="1" visible="no" active="yes"/>
-<layer number="212" name="212bmp" color="7" fill="1" visible="no" active="yes"/>
-<layer number="213" name="213bmp" color="7" fill="1" visible="no" active="yes"/>
-<layer number="214" name="214bmp" color="7" fill="1" visible="no" active="yes"/>
-<layer number="215" name="215bmp" color="7" fill="1" visible="no" active="yes"/>
-<layer number="216" name="216bmp" color="7" fill="1" visible="no" active="yes"/>
-<layer number="217" name="217bmp" color="18" fill="1" visible="no" active="no"/>
-<layer number="218" name="218bmp" color="19" fill="1" visible="no" active="no"/>
-<layer number="219" name="219bmp" color="20" fill="1" visible="no" active="no"/>
-<layer number="220" name="220bmp" color="21" fill="1" visible="no" active="no"/>
-<layer number="221" name="221bmp" color="22" fill="1" visible="no" active="no"/>
-<layer number="222" name="222bmp" color="23" fill="1" visible="no" active="no"/>
-<layer number="223" name="223bmp" color="24" fill="1" visible="no" active="no"/>
-<layer number="224" name="224bmp" color="25" fill="1" visible="no" active="no"/>
-<layer number="250" name="Descript" color="3" fill="1" visible="no" active="no"/>
-<layer number="251" name="SMDround" color="12" fill="11" visible="no" active="no"/>
-<layer number="254" name="cooling" color="7" fill="1" visible="no" active="yes"/>
 </layers>
 <board>
@@
 <param name="mdViaViaSameLayer" value="8mil"/>
 <param name="mnLayersViaInSmd" value="2"/>
-<param name="mdCopperDimension" value="40mil"/>
+<param name="mdCopperDimension" value="30mil"/>
 <param name="mdDrill" value="6mil"/>
 <param name="mdSmdStop" value="0mil"/>
@@
 <element name="C126" library="Parts for D-DAQ" package="SMD-0603" value="0.1uF" x="42.338625" y="33.670875" rot="R180"/>
 <element name="C127" library="Parts for D-DAQ" package="SMD-0603" value="0.1uF" x="43.005375" y="33.7185" rot="MR180"/>
-<element name="5V-TOGGLE-1" library="Parts for D-DAQ" package="SOP-4--CPC1117N" value="NC SSR" x="40.07235" y="17.99069375" rot="MR315"/>
-<element name="3.3V-TOGGLE-1" library="Parts for D-DAQ" package="SOP-4--CPC1017N" value="NO SSR" x="39.310353125" y="12.25935" rot="MR315"/>
+<element name="5V-TOGGLE-1" library="Parts for D-DAQ" package="SOP-4-NC" value="NC SSR" x="40.07235" y="17.99069375" rot="MR315"/>
+<element name="3.3V-TOGGLE-1" library="Parts for D-DAQ" package="SOP-4-NO" value="NO SSR" x="39.310353125" y="12.25935" rot="MR315"/>
 <element name="C118" library="Parts for D-DAQ" package="SMD-0603" value="0.1uF" x="57.87254375" y="22.43954375" rot="R135"/>
 <element name="C117" library="Parts for D-DAQ" package="SMD-0603" value="0.1uF" x="58.1025" y="29.62275" rot="R315"/>
@@
 <element name="R127" library="Parts for D-DAQ" package="SMD-0603" value="10k" x="61.1505" y="27.33675" rot="R180"/>
 <element name="R135" library="Parts for D-DAQ" package="SMD-0603" value="10k" x="69.43725" y="19.90725" rot="R135"/>
-<element name="5V-TOGGLE-2" library="Parts for D-DAQ" package="SOP-4--CPC1117N" value="NC SSR" x="88.5825" y="15.71625" rot="MR0"/>
-<element name="3.3V-TOGGLE-2" library="Parts for D-DAQ" package="SOP-4--CPC1017N" value="NO SSR" x="81.3435" y="15.71625" rot="MR0"/>
+<element name="5V-TOGGLE-2" library="Parts for D-DAQ" package="SOP-4-NC" value="NC SSR" x="88.5825" y="15.71625" rot="MR0"/>
+<element name="3.3V-TOGGLE-2" library="Parts for D-DAQ" package="SOP-4-NO" value="NO SSR" x="81.3435" y="15.71625" rot="MR0"/>
 <element name="MMA8652FC" library="Parts for D-DAQ" package="QFN-12" value="Accelerometer" x="43.14825" y="40.1955" rot="R90"/>
 <element name="R140" library="Parts for D-DAQ" package="SMD-0603" value="1.4k" x="46.101" y="41.529"/>
@@
 <element name="Y1" library="Parts for D-DAQ" package="3.2X2.5MM" value="XTC7009" x="53.482875" y="38.95725" rot="MR180"/>
 <element name="C1" library="Parts for D-DAQ" package="SMD-0603" value="10nF" x="53.49921875" y="38.052378125" rot="R90"/>
-<element name="5V-REG" library="Parts for D-DAQ" package="SOT-223-5" value="ZLDO1117-5.0" x="10.00125" y="41.91" rot="R180"/>
+<element name="5V-REG" library="Parts for D-DAQ" package="SOT-223-4" value="ZLDO1117-5.0" x="10.00125" y="41.91" rot="R180"/>
 <element name="MAIN-SMPS" library="Parts for D-DAQ" package="QFN-14" value="MP2209" x="16.09725" y="21.43125" rot="R270"/>
 <element name="L1" library="Parts for D-DAQ" package="7443551XXX" value="7.6uH" x="15.621" y="6.477"/>
@@
 <element name="R20" library="Parts for D-DAQ" package="SMD-0603" value="100" x="79.91475" y="10.8585" rot="MR180"/>
 <element name="JTAG" library="Parts for D-DAQ" package="HEADER-X4" value="HEADER-X4" x="46.76775" y="28.432125" rot="R90"/>
-<element name="5V-TOGGLE-5" library="Parts for D-DAQ" package="SOP-4--CPC1117N" value="NC SSR" x="41.005125" y="26.431875" rot="R180"/>
-<element name="3.3V-TOGGLE-5" library="Parts for D-DAQ" package="SOP-4--CPC1017N" value="NO SSR" x="42.624375" y="27.574875" rot="MR180"/>
+<element name="5V-TOGGLE-5" library="Parts for D-DAQ" package="SOP-4-NC" value="NC SSR" x="41.005125" y="26.431875" rot="R180"/>
+<element name="3.3V-TOGGLE-5" library="Parts for D-DAQ" package="SOP-4-NO" value="NO SSR" x="42.624375" y="27.574875" rot="MR180"/>
 <element name="R15" library="Parts for D-DAQ" package="SMD-0603" value="100" x="43.434" y="30.099" rot="R270"/>
 <element name="C9" library="Parts for D-DAQ" package="SMD-0603" value="4.7uF" x="39.624" y="30.6705" rot="R135"/>
