File: Design Files/D-DAQ Mainboard.sch (EAGLE design)
At the start: 117 parts, among them Y1 16.368 MHz, Y2 DS1099

Commit message: Update to Proto v3.6. Please visit the following for details: http://hackaday.io/project/964/log/4782
Parts:
- removed R13: 10k, resistor:R-US_R0603
- added C10, C11, C9: 4.7uF, Parts for D-DAQ:C-0603
- 10&11, 12&13, 4&5, 8&9, IMP.: device Parts for DC MF Gauge:105133-0001 -> Parts for D-DAQ:105133-0001
- 14V-REG: device Parts for DC MF Gauge:TL1963A-33DCQ -> Parts for D-DAQ:TL1963A-33DCQ
- 2.8V: device Parts for DC MF Gauge:TC1016 -> Parts for D-DAQ:TC1016
- 3.3V-TOGGLE-1, 3.3V-TOGGLE-2, 3.3V-TOGGLE-5: device Parts for DC MF Gauge:CPC1017N -> Parts for D-DAQ:CPC1017N
- 5V-REG: device Parts for DC MF Gauge:ZLDO1117-ADJ -> Parts for D-DAQ:ZLDO1117-ADJ
- 5V-TOGGLE-1, 5V-TOGGLE-2, 5V-TOGGLE-5: device Parts for DC MF Gauge:CPC1117N -> Parts for D-DAQ:CPC1117N
- 6&7+: device Parts for DC MF Gauge:47589-0001 -> Parts for D-DAQ:47589-0001
- AS7C31026B: device Parts for DC MF Gauge:AS7C31026B-12TC -> Parts for D-DAQ:AS7C31026B-12TC
- AUX-PRESS: device con-molex-alt:PC-1771101 -> Parts for D-DAQ:PC-1771101
- C1, C117, C118, C119, C121, C122, C123, C124, C125, C126, C127, C2, C4, C5, C6, C7, C8: device resistor:C-USC0603K -> Parts for D-DAQ:C-0603
- C1.1, C1.2: device resistor:C-USC1206 -> Parts for D-DAQ:C-1812
- C2.1, C2.2, C21, C22, C3, C31: device resistor:C-USC1206 -> Parts for D-DAQ:C-1206
- CAN-BUS, DATA: device Parts for DC MF Gauge:UE25-BE55-10H -> Parts for D-DAQ:UE25-BE55-10H
- D4: device Parts for D-DAQ:TFZ-DIODE -> Parts for D-DAQ:TFZ20B
- DISP-1, DISP-2, DISP-3: value DP3AR020SU32JQ1-STANDARD -> (none); device con-molex-alt:DP3AR020SU32JQ1-STANDARD -> Parts for D-DAQ:DP3R020SU32JQ
- EGT, POWER: device Parts for DC MF Gauge:1702610 -> Parts for D-DAQ:1702610
- EGT-AMP: device Parts for DC MF Gauge:MAX4239 -> Parts for D-DAQ:MAX4239
- F0, F1, F10, F11, F12, F13, F14, F2, F3, F4, F5, F6, F7, F8, F9, R1, R10, R11, R12, R127, R129, R130, R131, R132, R133, R135, R136, R138, R139, R14, R140, R141, R142, R145, R146, R147, R15, R2, R20, R21, R3, R31, R32, R4, R5, R6, R7, R8, R9: device resistor:R-US_R0603 -> Parts for D-DAQ:R-0603
- JTAG: value (none) -> HEADER-X4; device pinhead:PINHD-1X4 -> Parts for D-DAQ:HEADER-X4
- L1: device Parts for DC MF Gauge:WE-INDUCTOR -> Parts for D-DAQ:WE-INDUCTOR
- LATCH-HIGH, LATCH-LOW: device Parts for DC MF Gauge:74LVC573A -> Parts for D-DAQ:74LVC573A
- MAIN-SMPS: device Parts for DC MF Gauge:MP2209 -> Parts for D-DAQ:MP2209
- MICRO-SD: device Parts for DC MF Gauge:MICRO-SD-SLOT -> Parts for D-DAQ:MICRO-SD-SLOT
- MMA8652FC: device Parts for DC MF Gauge:MMA8491Q -> Parts for D-DAQ:MMA8491Q
- MPL3115A101: device Parts for DC MF Gauge:MPL3115A2 -> Parts for D-DAQ:MPL3115A2
- NBPLANN100PAUNV: device Parts for DC MF Gauge:NBP-SENSORS -> Parts for D-DAQ:NBP-SENSORS
- PIC32MX: device Parts for DC MF Gauge:PIC32MX795F512L-80I/PT -> Parts for D-DAQ:PIC32MX795F512L-80I/PT
- SC18IS602B: device Parts for DC MF Gauge:SC18IS602B -> Parts for D-DAQ:SC18IS602B
- Y1: value 16.368 MHz -> XTC7009; device Parts for DC MF Gauge:XTC7009 -> Parts for D-DAQ:XTC7009
- Y2: device Parts for DC MF Gauge:DS1099 -> Parts for D-DAQ:DS1099
Connections:
- removed net OE0: R13.1, Y2.OE0
- new net BOOST-SSR: 3.3V-TOGGLE-2.C+, 5V-TOGGLE-2.C-, C11.2
- new net USB-SSR: 3.3V-TOGGLE-1.C+, 5V-TOGGLE-1.C-, C10.2
- net 100-PSI-SENSOR-RES: no longer 3.3V-TOGGLE-2.C+
- net 12V-INPUT: now also D2.A; no longer D2.P$1
- net 14V-INPUT: now also D3.C; no longer D3.P$2
- net 3.3V-RAIL: now also 3.3V-TOGGLE-1.L1, 3.3V-TOGGLE-2.L1; no longer 3.3V-TOGGLE-1.L2, 3.3V-TOGGLE-2.L2
- net 5V-RAIL: now also 5V-TOGGLE-1.L2, Y2.OE0; no longer 5V-TOGGLE-1.L1
- net AUTO-DETECT: no longer 3.3V-TOGGLE-1.C+
- net BOOST-PWR: now also 3.3V-TOGGLE-2.L2; no longer 3.3V-TOGGLE-2.L1
- net CP-PUMP: now also D2.C, D3.A; no longer D2.P$2, D3.P$1
- net EGT-NEG-IN: now also R136.1; no longer R136.2
- net EGT-SHTDWN: now also R132.2; no longer R132.1
- net GND: now also C10.1, C11.1, C9.2, D1.A, R132.1, R136.2; no longer 5V-TOGGLE-1.C-, 5V-TOGGLE-2.C-, D1.P$1, R13.2, R132.2, R136.1
- net ICSP-SSR: now also C9.1
- net PWR-GND: now also D1.C; no longer D1.P$2
- net USB-PWR: now also 3.3V-TOGGLE-1.L2, 5V-TOGGLE-1.L1; no longer 3.3V-TOGGLE-1.L1, 5V-TOGGLE-1.L2
Other:
- note added: "Schematic Capture for D-DAQ Version: Proto v3.6 Released Under CERN OHL v1.2"
- moved on the sheet: R132, R136

Commit message: v3.6.1 No major changes, just cleanup and moving to Eagle v6.6 files
Changed lines of the file:
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@@
 <?xml version="1.0" encoding="utf-8"?>
 <!DOCTYPE eagle SYSTEM "eagle.dtd">
-<eagle version="6.4">
+<eagle version="6.6.0">
 <drawing>
 <settings>
@@
 <layer number="51" name="tDocu" color="14" fill="1" visible="no" active="no"/>
 <layer number="52" name="bDocu" color="7" fill="1" visible="no" active="no"/>
-<layer number="53" name="tGND_GNDA" color="7" fill="9" visible="no" active="no"/>
-<layer number="54" name="bGND_GNDA" color="1" fill="9" visible="no" active="no"/>
-<layer number="56" name="wert" color="7" fill="1" visible="no" active="no"/>
 <layer number="91" name="Nets" color="2" fill="1" visible="yes" active="yes"/>
 <layer number="92" name="Busses" color="1" fill="1" visible="yes" active="yes"/>
@@
 <layer number="97" name="Info" color="7" fill="1" visible="yes" active="yes"/>
 <layer number="98" name="Guide" color="6" fill="1" visible="yes" active="yes"/>
-<layer number="99" name="SpiceOrder" color="5" fill="1" visible="no" active="no"/>
-<layer number="100" name="Muster" color="7" fill="1" visible="no" active="no"/>
-<layer number="101" name="Patch_Top" color="12" fill="4" visible="no" active="yes"/>
-<layer number="102" name="Vscore" color="7" fill="1" visible="no" active="yes"/>
-<layer number="103" name="tMap" color="7" fill="1" visible="no" active="yes"/>
-<layer number="104" name="Name" color="16" fill="1" visible="no" active="yes"/>
-<layer number="105" name="tPlate" color="7" fill="1" visible="no" active="yes"/>
-<layer number="106" name="bPlate" color="7" fill="1" visible="no" active="yes"/>
-<layer number="107" name="Crop" color="7" fill="1" visible="no" active="yes"/>
-<layer number="116" name="Patch_BOT" color="9" fill="4" visible="no" active="yes"/>
-<layer number="121" name="_tsilk" color="7" fill="1" visible="no" active="yes"/>
-<layer number="122" name="_bsilk" color="7" fill="1" visible="no" active="yes"/>
-<layer number="125" name="_tNames" color="7" fill="1" visible="no" active="yes"/>
-<layer number="144" name="Drill_legend" color="7" fill="1" visible="no" active="yes"/>
-<layer number="151" name="HeatSink" color="7" fill="1" visible="no" active="yes"/>
-<layer number="200" name="200bmp" color="1" fill="10" visible="no" active="yes"/>
-<layer number="201" name="201bmp" color="2" fill="10" visible="no" active="yes"/>
-<layer number="202" name="202bmp" color="3" fill="10" visible="no" active="yes"/>
-<layer number="203" name="203bmp" color="4" fill="10" visible="no" active="yes"/>
-<layer number="204" name="204bmp" color="5" fill="10" visible="no" active="yes"/>
-<layer number="205" name="205bmp" color="6" fill="10" visible="no" active="yes"/>
-<layer number="206" name="206bmp" color="7" fill="10" visible="no" active="yes"/>
-<layer number="207" name="207bmp" color="8" fill="10" visible="no" active="yes"/>
-<layer number="208" name="208bmp" color="9" fill="10" visible="no" active="yes"/>
-<layer number="209" name="209bmp" color="7" fill="1" visible="no" active="yes"/>
-<layer number="210" name="210bmp" color="7" fill="1" visible="no" active="yes"/>
-<layer number="211" name="211bmp" color="7" fill="1" visible="no" active="yes"/>
-<layer number="212" name="212bmp" color="7" fill="1" visible="no" active="yes"/>
-<layer number="213" name="213bmp" color="7" fill="1" visible="no" active="yes"/>
-<layer number="214" name="214bmp" color="7" fill="1" visible="no" active="yes"/>
-<layer number="215" name="215bmp" color="7" fill="1" visible="no" active="yes"/>
-<layer number="216" name="216bmp" color="7" fill="1" visible="no" active="yes"/>
-<layer number="217" name="217bmp" color="18" fill="1" visible="no" active="no"/>
-<layer number="218" name="218bmp" color="19" fill="1" visible="no" active="no"/>
-<layer number="219" name="219bmp" color="20" fill="1" visible="no" active="no"/>
-<layer number="220" name="220bmp" color="21" fill="1" visible="no" active="no"/>
-<layer number="221" name="221bmp" color="22" fill="1" visible="no" active="no"/>
-<layer number="222" name="222bmp" color="23" fill="1" visible="no" active="no"/>
-<layer number="223" name="223bmp" color="24" fill="1" visible="no" active="no"/>
-<layer number="224" name="224bmp" color="25" fill="1" visible="no" active="no"/>
-<layer number="250" name="Descript" color="3" fill="1" visible="no" active="no"/>
-<layer number="251" name="SMDround" color="12" fill="11" visible="no" active="no"/>
-<layer number="254" name="cooling" color="7" fill="1" visible="no" active="yes"/>
 </layers>
 <schematic xreflabel="%F%N/%S.%C%R" xrefpart="/%S.%C%R">
@@
 <part name="C127" library="Parts for D-DAQ" deviceset="C-" device="0603" value="0.1uF"/>
 <part name="GND-PIC6" library="supply1" deviceset="GNDA" device="" value=""/>
-<part name="5V-TOGGLE-1" library="Parts for D-DAQ" deviceset="CPC1117N" device="" value="NC SSR"/>
-<part name="3.3V-TOGGLE-1" library="Parts for D-DAQ" deviceset="CPC1017N" device="" value="NO SSR"/>
+<part name="5V-TOGGLE-1" library="Parts for D-DAQ" deviceset="CPC1?17N" device="1" value="NC SSR"/>
+<part name="3.3V-TOGGLE-1" library="Parts for D-DAQ" deviceset="CPC1?17N" device="0" value="NO SSR"/>
 <part name="C118" library="Parts for D-DAQ" deviceset="C-" device="0603" value="0.1uF"/>
 <part name="C117" library="Parts for D-DAQ" deviceset="C-" device="0603" value="0.1uF"/>
@@
 <part name="R135" library="Parts for D-DAQ" deviceset="R-" device="0603" value="10k"/>
 <part name="GND-PIC3" library="supply1" deviceset="GNDA" device="" value=""/>
-<part name="5V-TOGGLE-2" library="Parts for D-DAQ" deviceset="CPC1117N" device="" value="NC SSR"/>
-<part name="3.3V-TOGGLE-2" library="Parts for D-DAQ" deviceset="CPC1017N" device="" value="NO SSR"/>
+<part name="5V-TOGGLE-2" library="Parts for D-DAQ" deviceset="CPC1?17N" device="1" value="NC SSR"/>
+<part name="3.3V-TOGGLE-2" library="Parts for D-DAQ" deviceset="CPC1?17N" device="0" value="NO SSR"/>
 <part name="MMA8652FC" library="Parts for D-DAQ" deviceset="MMA8491Q" device="" value="Accelerometer"/>
 <part name="R140" library="Parts for D-DAQ" deviceset="R-" device="0603" value="1.4k"/>
@@
 <part name="Y1" library="Parts for D-DAQ" deviceset="XTC7009" device="" value="XTC7009"/>
 <part name="C1" library="Parts for D-DAQ" deviceset="C-" device="0603" value="10nF"/>
-<part name="5V-REG" library="Parts for D-DAQ" deviceset="ZLDO1117-ADJ" device="" value="ZLDO1117-5.0"/>
+<part name="5V-REG" library="Parts for D-DAQ" deviceset="ZLDO1117-" device="ADJ" value="ZLDO1117-5.0"/>
 <part name="MAIN-SMPS" library="Parts for D-DAQ" deviceset="MP2209" device=""/>
 <part name="L1" library="Parts for D-DAQ" deviceset="WE-INDUCTOR" device="" value="7.6uH"/>
@@
 <part name="R20" library="Parts for D-DAQ" deviceset="R-" device="0603" value="100"/>
 <part name="JTAG" library="Parts for D-DAQ" deviceset="HEADER-X?" device="4"/>
-<part name="5V-TOGGLE-5" library="Parts for D-DAQ" deviceset="CPC1117N" device="" value="NC SSR"/>
-<part name="3.3V-TOGGLE-5" library="Parts for D-DAQ" deviceset="CPC1017N" device="" value="NO SSR"/>
+<part name="5V-TOGGLE-5" library="Parts for D-DAQ" deviceset="CPC1?17N" device="1" value="NC SSR"/>
+<part name="3.3V-TOGGLE-5" library="Parts for D-DAQ" deviceset="CPC1?17N" device="0" value="NO SSR"/>
 <part name="R15" library="Parts for D-DAQ" deviceset="R-" device="0603" value="100"/>
 <part name="D1" library="Parts for D-DAQ" deviceset="S07D" device=""/>

Commit message: update component values
Parts:
- 2.8V: value TC1016 -> TC1016-2.8VCTTR
- C1.1, C1.2: value 47uF -> 22uF
- C124, C125, C2: value 10uF -> 22uF
- C2.1, C2.2, C22: value 4.7uF -> 10uF; device Parts for D-DAQ:C-1206 -> Parts for D-DAQ:C-1210
- C21: value 47uF -> 4.7uF
- C31: device Parts for D-DAQ:C-1206 -> Parts for D-DAQ:C-1210
- CAN-BUS, DATA: value Mini USB -> UE25BE5510H
- D1: value S07D -> S07D-GS08
- D4: value TFZ20B -> TFZGTR20B; device Parts for D-DAQ:TFZ20B -> Parts for D-DAQ:TFZGTR20B
- DISP-1, DISP-2, DISP-3: value (none) -> Standard
- MICRO-SD: value SCHA4B0400 -> 47579-0001
- R14: value 34 -> 33.2
- renumbered 3.3V-TOGGLE-5 to 3.3V-TOGGLE-3, 5V-TOGGLE-5 to 5V-TOGGLE-3
Connections:
- net 12V-FB: now also R1.2, R2.1; no longer R1.1, R2.2
- net 14V-RAIL: now also C31.2; no longer C31.1
- net 3.3V-RAIL: now also R1.1; no longer R1.2
- net CHARG-CAPS: now also C2.1.1; no longer C2.1.2
- net CP-PUMP: now also C2.1.2; no longer C2.1.1
- net GND: now also C31.1, R2.2; no longer C31.2, R2.1
Other:
- note added: "Schematic Capture for D-DAQ Version: Proto v3.6.5 Released Under CERN OHL v1.2"
- note removed: "Schematic Capture for D-DAQ Version: Proto v3.6 Released Under CERN OHL v1.2"
- moved on the sheet: R1, R2

Commit message: Updating to Proto 4
Parts:
- removed 10&11, 12&13, 4&5, 8&9, IMP.: Micro USB, Parts for D-DAQ:105133-0001
- removed 14V-REG: TL1963A-33DCQ, Parts for D-DAQ:TL1963A-33DCQ
- removed 2.8V: TC1016-2.8VCTTR, Parts for D-DAQ:TC1016
- removed 3.3V-TOGGLE-1, 3.3V-TOGGLE-2, 3.3V-TOGGLE-3: NO SSR, Parts for D-DAQ:CPC1017N
- removed 5V-REG: ZLDO1117-5.0, Parts for D-DAQ:ZLDO1117-ADJ
- removed 5V-TOGGLE-1, 5V-TOGGLE-2, 5V-TOGGLE-3: NC SSR, Parts for D-DAQ:CPC1117N
- removed 6&7+: Micro USB, Parts for D-DAQ:47589-0001
- removed AS7C31026B: 1 Mbit SRAM, Parts for D-DAQ:AS7C31026B-12TC
- removed AUX-PRESS: PC-1771101, Parts for D-DAQ:PC-1771101
- removed C1, C6: 10nF, Parts for D-DAQ:C-0603
- removed C1.1, C1.2: 22uF, Parts for D-DAQ:C-1812
- removed C10, C11, C123, C9: 4.7uF, Parts for D-DAQ:C-0603
- removed C117, C118, C119, C121, C122, C126, C127, C5, C7, C8: 0.1uF, Parts for D-DAQ:C-0603
- removed C124, C125, C2: 22uF, Parts for D-DAQ:C-0603
- removed C2.1, C2.2, C22, C31: 10uF, Parts for D-DAQ:C-1210
- removed C21: 4.7uF, Parts for D-DAQ:C-1206
- removed C3: 47uF, Parts for D-DAQ:C-1206
- removed C4: 1uF, Parts for D-DAQ:C-0603
- removed CAN-BUS, DATA: UE25BE5510H, Parts for D-DAQ:UE25-BE55-10H
- removed D1: S07D-GS08, Parts for D-DAQ:S07D
- removed D2, D3: PMEG2010ER, Parts for D-DAQ:S07D
- removed D4: TFZGTR20B, Parts for D-DAQ:TFZGTR20B
- removed EGT-AMP: MAX4239, Parts for D-DAQ:MAX4239
- removed F0, F1, F10, F11, F12, F13, F14, F2, F3, F4, F5, F6, F7, F8, F9: 470, Parts for D-DAQ:R-0603
- removed JTAG: HEADER-X4, Parts for D-DAQ:HEADER-X4
- removed L1: 7.6uH, Parts for D-DAQ:WE-INDUCTOR
- removed LATCH-HIGH, LATCH-LOW: Octal D-Latch, Parts for D-DAQ:74LVC573A
- removed MAIN-SMPS: MP2209, Parts for D-DAQ:MP2209
- removed MICRO-SD: 47579-0001, Parts for D-DAQ:MICRO-SD-SLOT
- removed MMA8652FC: Accelerometer, Parts for D-DAQ:MMA8491Q
- removed MPL3115A101: Baro & Temp, Parts for D-DAQ:MPL3115A2
- removed NBPLANN100PAUNV: Boost, Parts for D-DAQ:NBP-SENSORS
- removed PIC32MX: 795F512L-80V/PT, Parts for D-DAQ:PIC32MX795F512L-80I/PT
- removed POWER: 1702610, Parts for D-DAQ:1702610
- removed R1: 499k, Parts for D-DAQ:R-0603
- removed R10, R12, R127, R129, R130, R132, R135, R138, R139, R142, R145, R146, R147, R6, R7, R8, R9: 10k, Parts for D-DAQ:R-0603
- removed R11, R136, R140, R141: 1.4k, Parts for D-DAQ:R-0603
- removed R131: 255, Parts for D-DAQ:R-0603
- removed R133, R3, R5: 100k, Parts for D-DAQ:R-0603
- removed R14: 33.2, Parts for D-DAQ:R-0603
- removed R15, R20, R21: 100, Parts for D-DAQ:R-0603
- removed R2: 158k, Parts for D-DAQ:R-0603
- removed R31: 3.01k, Parts for D-DAQ:R-0603
- removed R32: 30.9k, Parts for D-DAQ:R-0603
- removed R4: 10, Parts for D-DAQ:R-0603
- removed SC18IS602B: I2C to SPI, Parts for D-DAQ:SC18IS602B
- removed Y1: XTC7009, Parts for D-DAQ:XTC7009
- removed Y2: DS1099, Parts for D-DAQ:DS1099
- added 12V, 14V, 3.3V, 3.3V-2, 3.3V-3, 5V, TP1, TP2, TP3, TP4, TP5, TP6, TP7: TP-0463, Parts for D-DAQ:TP-0463
- added AUX: PC-3-1771101, Parts for D-DAQ:PC-3-1771101
- added C101, C601, C802, C803: 0.1uF, Parts for D-DAQ:C-0603
- added C102, C801: 10uF, Parts for D-DAQ:C-0805
- added C103: 10nF, Parts for D-DAQ:C-0603
- added C901, C902, C903: 4.7uF, Parts for D-DAQ:C-0603
- added CAN, USB: UE25BE5510H, Parts for D-DAQ:UE25-BE55-10H
- added CF101, CF102, CF103: (no value), Parts for D-DAQ:NMF21PS
- added F900, F901, F902, F903, F904, F905, F908, F909, F910, F911, F912, F913: 470, Parts for D-DAQ:F-0603
- added FB601, FB603, FB604, FB605, FB606, FB607, FB608, FB901: 470, Parts for D-DAQ:FB-0603
- added IMP-1&2, IMP-3, P-10&11, P-12&13, P-4&5, P-8&9: Micro USB, Parts for D-DAQ:105133-0001
- added K1001, K1003, K1005: NC SSR, Parts for D-DAQ:CPC1117N
- added K1002, K1004, K1006, K1007, K1008: NO SSR, Parts for D-DAQ:CPC1017N
- added LED101: Yellow, Parts for D-DAQ:LED-0603
- added LED901: Red, Parts for D-DAQ:LED-0603
- added MEM1001: IS61WV25616ALL, Parts for D-DAQ:IS61WV25616ALL
- added R101, R102, R103, R105, R106, R107, R202, R716, R717, R718, R719, R803, R804, R805, R806, R903, R905: 10k, Parts for D-DAQ:R-0603
- added R104: 470, Parts for D-DAQ:R-0603
- added R201, R801, R802, R901: 1.4k, Parts for D-DAQ:R-0603
- added R700, R701, R702, R703, R704, R705, R706, R707, R708, R709, R710, R711, R712, R713, R714, R715: 140, Parts for D-DAQ:R-0402
- added R902: 100k, Parts for D-DAQ:R-0603
- added R904: 255, Parts for D-DAQ:R-0603
- added R906, R907, R908, R909: 100, Parts for D-DAQ:R-0603
- added U1001: 795F512L-80V/PT, Parts for D-DAQ:PIC32MX795F512L-80I/PF
- added U1002, U1003: Octal D-Latch, Parts for D-DAQ:74LVC573A
- added U1004: Baro & Temp, Parts for D-DAQ:MPL3115A2
- added U1005: Boost, Parts for D-DAQ:NBP-SENSORS
- added U1006: Accelerometer, Parts for D-DAQ:MMA8491Q
- added U1007: MAX4239, Parts for D-DAQ:MAX4239
- added U1008: NXP-74HC165, Parts for D-DAQ:NXP-74HC165
- added X1: (no value), Parts for D-DAQ:MOLEX-87760-0816
- added X3: MOLEX-87760-1216", Parts for D-DAQ:MOLEX-87760-1216"
- added Y1001: XTC7009, Parts for D-DAQ:XTC7009
- EGT: value 1702610 -> (none); device Parts for D-DAQ:1702610 -> Parts for D-DAQ:PC-2-1702610
Connections:
- removed net 100-PSI-SENSOR-RES: 5V-TOGGLE-2.C+, R20.2
- removed net 12V-BS: C5.1, MAIN-SMPS.BS
- removed net 12V-ENABLE: MAIN-SMPS.EN, R3.1
- removed net 12V-FB: MAIN-SMPS.FB, R1.2, R2.1
- removed net 12V-OK: MAIN-SMPS.POK, R5.2
- removed net 12V-SS: C6.1, MAIN-SMPS.SS
- removed net 12V-SW: C5.2, L1.P$1, MAIN-SMPS.SW1, MAIN-SMPS.SW2
- removed net 12V-VCC: C4.2, MAIN-SMPS.VCC, R3.2, R4.1, R5.1
- removed net 14V-12V-DIVIDER: F0.2, R10.2, R11.2
- removed net 14V-ADJ: 14V-REG.ADJ, R31.2, R32.1
- removed net 14V-INPUT: 14V-REG.SHDN, 14V-REG.VIN, C2.2.1, D3.C, R14.1
- removed net 3.3-&-5V-TOGGLE1: PIC32MX.GPIO-A9, R21.1
- removed net 3.3-&-5V-TOGGLE2: PIC32MX.GPIO-A10, R20.1
- removed net 3.3V-RAIL: 2.8V.SHDN, 2.8V.V-IN, 3.3V-TOGGLE-1.L1, 3.3V-TOGGLE-2.L1, AS7C31026B.VCC-1, AS7C31026B.VCC-2, C117.1, C118.2, C119.1, C122.1, C123.2, C125.1, C126.2, C2.2, C3.2, DISP-1.4, DISP-2.4, DISP-3.4, IMP..1, L1.P$2, LATCH-HIGH.VCC, LATCH-LOW.VCC, MICRO-SD.VDD, MMA8652FC.VDD, MPL3115A101.VDD, MPL3115A101.VDDIO, PIC32MX.AVDD, PIC32MX.V-USB-3.3, PIC32MX.VDD-1, PIC32MX.VDD-2, PIC32MX.VDD-3, PIC32MX.VDD-4, PIC32MX.VDD-5, PIC32MX.VDD-6, R1.1, R12.1, R138.2, R140.2, R141.1, R15.1, R8.2, R9.1, SC18IS602B.VDD
- removed net 5V-ADJ: 5V-REG.(GND), C22.2
- removed net 6&7-PIN1: 3.3V-TOGGLE-3.L1, 5V-TOGGLE-3.L1, 6&7+.1
- removed net A0-PD: R7.2, SC18IS602B.A0
- removed net A1-PD: R6.1, SC18IS602B.A1
- removed net A2-PU: R8.1, SC18IS602B.A2
- removed net ADD-0: AS7C31026B.A0, LATCH-LOW.7Q
- removed net ADD-1: AS7C31026B.A1, LATCH-LOW.6Q
- removed net ADD-10: AS7C31026B.A10, LATCH-HIGH.5Q
- removed net ADD-11: AS7C31026B.A11, LATCH-HIGH.4Q
- removed net ADD-12: AS7C31026B.A12, LATCH-HIGH.3Q
- removed net ADD-13: AS7C31026B.A13, LATCH-HIGH.2Q
- removed net ADD-14: AS7C31026B.A14, LATCH-HIGH.1Q
- removed net ADD-15: AS7C31026B.A15, LATCH-HIGH.0Q
- removed net ADD-2: AS7C31026B.A2, LATCH-LOW.5Q
- removed net ADD-3: AS7C31026B.A3, LATCH-LOW.4Q
- removed net ADD-4: AS7C31026B.A4, LATCH-LOW.3Q
- removed net ADD-5: AS7C31026B.A5, LATCH-LOW.2Q
- removed net ADD-6: AS7C31026B.A6, LATCH-LOW.1Q
- removed net ADD-7: AS7C31026B.A7, LATCH-LOW.0Q
- removed net ADD-8: AS7C31026B.A8, LATCH-HIGH.7Q
- removed net ADD-9: AS7C31026B.A9, LATCH-HIGH.6Q
- removed net AN2-OIL-PESS: F2.1, PIC32MX.AN-2
- removed net AN3-EGT: F3.2, PIC32MX.AN-3
- removed net AN6: 6&7+.2, F6.1
- removed net AN7: 6&7+.3, F7.2
- removed net AUTO-DETECT: 5V-TOGGLE-1.C+, R21.2
- removed net BARO-INT2: MPL3115A101.INT2, R139.1
- removed net CAN-BUS1: CAN-BUS.P$2, PIC32MX.CAN2-TX-ALT
- removed net CAN-BUS2: CAN-BUS.P$3, PIC32MX.CAN2-RX-ALT
- removed net CARD-DETECT: MICRO-SD.CD1, SC18IS602B.GPIO-0
- removed net CE: AS7C31026B.CE, R142.1
- removed net CHARG-CAPS: C2.1.1, Y2.OUT1
- removed net CP-PUMP: C2.1.2, D2.C, D3.A
- removed net CPS-INPUT: IMP..2, PIC32MX.INPUT-CAPTURE-1
- removed net CRYSTAL-OUT: PIC32MX.CLK-OUT/OSC2
- removed net DISP-1_HPD: DISP-1.6, PIC32MX.GPIO-C4
- removed net DISP-HPD2: DISP-2.6, PIC32MX.GPIO-C1
- removed net DISP-HPD3: DISP-3.6, PIC32MX.GPIO-F3
- removed net EGT-SHTDWN: EGT-AMP.SHDN, R132.2
- removed net GND: 10&11.5, 12&13.5, 14V-REG.GND, 14V-REG.TAB, 2.8V.GND, 3.3V-TOGGLE-1.C-, 3.3V-TOGGLE-2.C-, 4&5.5, 6&7+.5, 8&9.5, AS7C31026B.GND-1, AS7C31026B.GND-2, AUX-PRESS.P$2, C1.1.2, C1.2, C1.2.2, C10.1, C11.1, C117.2, C118.1, C119.2, C121.2, C122.2, C123.1, C124.1, C125.2, C126.1, C127.1, C2.1, C2.2.2, C21.2, C3.1, C31.1, C4.1, C6.2, C7.1, C8.2, C9.2, CAN-BUS.P$5, D1.A, D4.A, DATA.P$5, DISP-1.1, DISP-1.13, DISP-1.14, DISP-1.19, DISP-1.7, DISP-1.8, DISP-1.BL, DISP-1.BR, DISP-1.FL, DISP-1.FR, DISP-2.1, DISP-2.13, DISP-2.14, DISP-2.19, DISP-2.7, DISP-2.8, DISP-2.BL, DISP-2.BR, DISP-2.FL, DISP-2.FR, DISP-3.1, DISP-3.13, DISP-3.14, DISP-3.19, DISP-3.7, DISP-3.8, DISP-3.BL, DISP-3.BR, DISP-3.FL, DISP-3.FR, EGT-AMP.GND, IMP..5, LATCH-HIGH.GND, LATCH-LOW.GND, MAIN-SMPS.AGND, MAIN-SMPS.PGND1, MAIN-SMPS.PGND2, MICRO-SD.GND1, MICRO-SD.GND2, MICRO-SD.VSS, MMA8652FC.GND1, MMA8652FC.GND2, MPL3115A101.GND, NBPLANN100PAUNV.GND, PIC32MX.AVSS, PIC32MX.VSS-1, PIC32MX.VSS-2, PIC32MX.VSS-3, PIC32MX.VSS-4, PIC32MX.VSS-5, R11.1, R127.1, R129.2, R130.1, R132.1, R135.2, R136.2, R139.2, R142.2, R145.2, R146.2, R147.2, R2.2, R31.1, R6.2, R7.1, SC18IS602B.VSS, Y1.GNDA, Y1.GNDB, Y2.GND, Y2.OE1
- removed net HB: AS7C31026B.HB, R146.1
- removed net I2C-INT-BUS-PIN1: MPL3115A101.INT1, PIC32MX.GPIO-A6
- removed net I2C-INT-BUS-PIN2: PIC32MX.GPIO-A7
- removed net I2C-PIN1: MMA8652FC.SCL, MPL3115A101.SCL, PIC32MX.I2C-1-CLK, R140.1
- removed net I2C-PIN2: MMA8652FC.SDA, MPL3115A101.SDA, PIC32MX.I2C-1-DATA, R141.2
- removed net I2C-SD-PIN1: PIC32MX.I2C-2-CLK, SC18IS602B.SDC
- removed net I2C-SD-PIN2: PIC32MX.12C-2-DATA, SC18IS602B.SDA
- removed net ICSP-MCLR: 3.3V-TOGGLE-3.L2, C7.2, F14.2, R12.2
- removed net ICSP-TRIP: 3.3V-TOGGLE-3.C-, 6&7+.4
- removed net ICSP-TRIP-PWR: 5V-TOGGLE-3.C+, R15.2
- removed net LB: AS7C31026B.LB, R147.1
- removed net LNS-INPUT: IMP..3, PIC32MX.INPUT-CAPTURE-2
- removed net N$5: C121.1, MMA8652FC.BYP
- removed net OE: AS7C31026B.OE, R145.1
- removed net OSC-PWR: 2.8V.V-OUT, C1.1, Y1.VDD
- removed net OSC-SIG: PIC32MX.CLK-IN/OSC-1, Y1.OUT
- removed net PMA-CS2: DISP-3.16, PIC32MX.PMP-CS2
- removed net PMA-HL: LATCH-HIGH.LE, PIC32MX.PMA-LH
- removed net PMD-READ: PIC32MX.PMP-RD
- removed net PWM1: DISP-3.15, PIC32MX.PWM-1
- removed net PWM2: DISP-2.15, PIC32MX.PWM-2
- removed net PWM3: DISP-1.15, PIC32MX.PWM-3
- removed net PWM4: DISP-1.10, DISP-1.12, DISP-2.10, DISP-2.12, DISP-3.10, DISP-3.12, PIC32MX.PWM-4
- removed net PWR-GND: D1.C, POWER.R
- removed net SD-MISO: MICRO-SD.MISO, SC18IS602B.MISO
- removed net SD-MOSI: MICRO-SD.MOSI, SC18IS602B.MOSI
- removed net SD-PULL-DOWN: MICRO-SD.CD2, R9.2
- removed net SENSOR_PAIR_AN10: F10.2, PIC32MX.AN-10
- removed net SENSOR_PAIR_AN11: F11.1, PIC32MX.AN-11
- removed net SENSOR_PAIR_AN12: F12.2, PIC32MX.AN-12
- removed net SENSOR_PAIR_AN13: F13.1, PIC32MX.AN-13
- removed net SENSOR_PAIR_AN4: F4.1, PIC32MX.AN-4
- removed net SENSOR_PAIR_AN5: F5.2, PIC32MX.AN-5
- removed net SENSOR_PAIR_AN6: F6.2, PIC32MX.AN-6_/_ICSP-CLK
- removed net SENSOR_PAIR_AN7: F7.1, PIC32MX.AN-7_/_ICSP-DATA
- removed net SENSOR_PAIR_AN8: F8.2, PIC32MX.AN-8
- removed net SENSOR_PAIR_AN9: F9.1, PIC32MX.AN-9
- removed net SHUNT: D4.C, R14.2
- removed net SPI2-DATA: DISP-1.9, PIC32MX.SPI2-DO
- removed net SPI2-SS: PIC32MX.SPI2-SS, R135.1
- removed net SPI3-DATA: DISP-2.9, PIC32MX.SPI3-DO
- removed net SPI3-SS: PIC32MX.SPI3-SS, R129.1
- removed net SPI4-CLK: DISP-3.3, PIC32MX.SPI4-CLK
- removed net SPI4-DATA: DISP-3.9, PIC32MX.SPI4-DO
- removed net SPI4-SS: PIC32MX.SPI4-SS, R127.2
- removed net USB-PIN1: DATA.P$1, PIC32MX.V-USB-BUS
- removed net USB-PIN2: DATA.P$2, PIC32MX.USB-D-
- removed net USB-PIN3: DATA.P$3, PIC32MX.USB-D+
- new net 3.3V-RAIL-1: 3.3V-2.TP, CF101.1
- new net 3.3V-RAIL-2: 3.3V.TP, CF102.1, DISP-1.18, DISP-2.18, DISP-3.18, K1004.L1, U1008.VCC
- new net 3.3V-RAIL-3: 3.3V-3.TP, CF103.1
- new net 6&7-PIN-1: K1005.L1, K1006.L2, X1.P$6
- new net ACCEL-BYP: C803.1, U1006.BYP
- new net ADT-1: K1001.C+, R906.2
- new net ADT-2: K1003.C+, R907.2
- new net ADT-3: K1005.C+, R908.2
- new net ADT-4: K1007.C+, K1008.C+, R909.2
- new net AGND: AUX.P$2, C101.2, C601.1, C903.2, CF101.2@1, CF101.2@2, FB601.2, FB603.2, FB604.2, FB605.2, FB901.2, R901.1, R903.2, R905.2, U1001.AVSS, U1007.V-, X1.P$8
- new net ALT-INT: U1001.GPIO-C13, U1004.INT1
- new net AN2-EGT: F902.2, U1001.AN-2
- new net AN3-AUX-PRESS: F903.2, U1001.AN-3
- new net BARO-INT: R803.2, U1004.INT2
- new net BOOST-GND: FB901.1, U1005.GND
- new net BOOST-V-TOGGLE: R906.1, U1001.GPIO-E9
- new net CAN-BUS-1: CAN.P$2, U1001.CAN2-TX-ALT
- new net CAN-BUS-2: CAN.P$3, U1001.CAN2-RX-ALT
- new net CLEAN-3.3V-1: CF101.3, K1002.L1, R102.1, R103.1, R105.1, R106.1, R908.1
- new net CLEAN-3.3V-2: C101.1, C103.1, C801.1, CF102.3, R107.2, R801.1, R802.1, R804.1, TP6.TP, U1001.AVDD, U1001.V-USB-3.3, U1001.VDD-1, U1001.VDD-2, U1001.VDD-3, U1001.VDD-4, U1001.VDD-5, U1001.VDD-6, U1004.VDD, U1004.VDDIO, U1006.VDD, Y1001.VDD
- new net CLEAN-3.3V-3: CF103.3, IMP-1&2.1, IMP-3.1, MEM1001.VCC-1, MEM1001.VCC-2, R805.1, R806.1, U1002.VCC, U1003.VCC, X3.P$7
- new net DGND: C102.2, C103.2, C801.2, C802.1, C803.2, C901.1, C902.1, CAN.P$5, CF102.2@1, CF102.2@2, CF103.2@1, CF103.2@2, DISP-1.1, DISP-1.13, DISP-1.14, DISP-1.19, DISP-1.7, DISP-1.8, DISP-1.BL, DISP-1.BR, DISP-1.FL, DISP-1.FR, DISP-2.1, DISP-2.13, DISP-2.14, DISP-2.19, DISP-2.7, DISP-2.8, DISP-2.BL, DISP-2.BR, DISP-2.FL, DISP-2.FR, DISP-3.1, DISP-3.13, DISP-3.14, DISP-3.19, DISP-3.7, DISP-3.8, DISP-3.BL, DISP-3.BR, DISP-3.FL, DISP-3.FR, FB606.2, FB607.2, FB608.1, K1002.C-, K1004.C-, LED101.2, MEM1001.GND-1, MEM1001.GND-2, R201.1, R716.2, R717.2, R718.2, R719.2, R803.1, TP7.TP, U1001.VSS-1, U1001.VSS-2, U1001.VSS-3, U1001.VSS-4, U1001.VSS-5, U1002.GND, U1003.GND, U1004.GND, U1006.GND1, U1006.GND2, U1008.-CE, U1008.GND, USB.P$5, X3.P$10, X3.P$12, X3.P$2, X3.P$4, X3.P$6, X3.P$8, Y1001.GNDA, Y1001.GNDB
- new net DISP1-HPD: DISP-1.17, R107.1, U1001.GPIO-F3
- new net DISP1-RS: DISP-1.5, U1001.SPI3-SS
- new net DISP2-HPD: DISP-2.17, R105.2, U1001.GPIO-E8
- new net DISP3-HPD: DISP-3.17, R102.2, U1001.GPIO-C4
- new net EGT-SHDN: R903.1, U1007.CRETN
- new net GND-FILTER: C601.2, FB608.2
- new net HB-PD: MEM1001.HB, R717.1
- new net I2C-CLK: R802.2, U1001.I2C-1-CLK, U1004.SCL, U1006.SCL
- new net I2C-DATA: R801.2, U1001.I2C-1-DATA, U1004.SDA, U1006.SDA
- new net ICSP-DETECT: K1006.C-, LED901.2, R106.2, U1001.GPIO-A9, X1.P$5
- new net ICSP-LED: K1007.C-, K1008.C-, LED901.1
- new net IMP-1: IMP-1&2.3, U1001.INPUT-CAPTURE-1
- new net IMP-2: IMP-1&2.2, U1001.INPUT-CAPTURE-2
- new net IMP-3: IMP-3.3, U1001.INPUT-CAPTURE-3
- new net INPUT-V-SENSE: F900.1, R201.2, R202.2
- new net LB-PD: MEM1001.LB, R716.1
- new net LOAD-AN6: K1007.L1, X1.P$1
- new net LOAD-AN7: K1008.L1, X1.P$3
- new net N$58: U1001.GPIO-A2
- new net NC$1: X1.P$7
- new net OE-PD: MEM1001.OE, R718.1
- new net OSCI: U1001.OSCI, Y1001.OUT
- new net PMA-LH: U1001.PMA-LH, U1003.LE
- new net PMD-0: MEM1001.I/O-0, R700.2, U1002.0D
- new net PMD-1: MEM1001.I/O-1, R701.2, U1002.1D
- new net PMD-10: MEM1001.I/O-10, R710.2, U1003.2D
- new net PMD-11: MEM1001.I/O-11, R711.2, U1003.3D
- new net PMD-12: MEM1001.I/O-12, R712.2, U1003.4D
- new net PMD-13: MEM1001.I/O-13, R713.2, U1003.5D
- new net PMD-15: MEM1001.I/O-15, R715.2, U1003.7D
- new net PMD-2: MEM1001.I/O-2, R702.2, U1002.2D
- new net PMD-3: MEM1001.I/O-3, R703.2, U1002.3D
- new net PMD-4: MEM1001.I/O-4, R704.2, U1002.4D
- new net PMD-5: MEM1001.I/O-5, R705.2, U1002.5D
- new net PMD-6: MEM1001.I/O-6, R706.2, U1002.6D
- new net PMD-7: MEM1001.I/O-7, R707.2, U1002.7D
- new net PMD-8: MEM1001.I/O-8, R708.2, U1003.0D
- new net PMD-9: MEM1001.I/O-9, R709.2, U1003.1D
- new net PMD14: R714.1, U1001.PMD-14
- new net PMP-READ: R719.1, U1001.PMRD/PMWR
- new net PWM-BL: DISP-1.16, DISP-1.6, DISP-2.16, DISP-2.6, DISP-3.16, DISP-3.6, U1001.PWM-4
- new net PWM1-WARN: DISP-1.3, U1001.PWM-3
- new net PWM2-WARN: DISP-2.3, U1001.PWM-2
- new net PWM3-WARN: DISP-3.3, U1001.PWM-1
- new net SD-CARD-DETECT: R805.2, U1001.GPIO-A3, X3.P$9
- new net SD-SPI-DI: U1001.GPIO-A7, X3.P$5
- new net SD-SPI-DO: U1001.GPIO-G15, X3.P$1
- new net SD-WRITE-PROTECT: R806.2, U1001.GPIO-C14, X3.P$11
- new net SENSOR-AN10: F910.2, U1001.AN-10
- new net SENSOR-AN11: F911.2, U1001.AN-11
- new net SENSOR-AN12: F912.2, U1001.AN-12
- new net SENSOR-AN13: F913.2, U1001.AN-13
- new net SENSOR-AN4: F904.1, U1001.AN-4
- new net SENSOR-AN5: F905.1, U1001.AN-5
- new net SENSOR-AN6: K1007.L2, U1001.AN-6_/_ICSP-CLK, X1.P$4
- new net SENSOR-AN7: K1008.L2, U1001.AN-7_/_ICSP-DATA, X1.P$2
- new net SENSOR-AN8: F908.2, U1001.AN-8
- new net SENSOR-AN9: F909.2, U1001.AN-9
- new net SGND-1: FB601.1, P-4&5.5
- new net SGND-3: FB603.1, P-8&9.5
- new net SGND-4: FB604.1, P-10&11.5
- new net SGND-5: FB605.1, P-12&13.5
- new net SGND-6: FB606.1, IMP-1&2.5
- new net SGND-7: FB607.1, IMP-3.5
- new net SHIFT-CS-LINE: U1001.GPIO-C1, U1008.-PL
- new net SOFT-PMP-CS2: U1001.GPIO-A6
- new net SPI1-CLK: DISP-1.15, U1001.SPI3-CLK
- new net SPI1-DO: DISP-1.9, U1001.SPI3-DO
- new net SPI2-DO: DISP-2.9, U1001.SPI4-DO
- new net SPI3-DO: DISP-3.9, U1001.SPI2-DO, U1008.DS
- new net SRAM-0: MEM1001.A0, U1002.0Q
- new net SRAM-1: MEM1001.A1, U1002.1Q
- new net SRAM-10: MEM1001.A10, U1003.2Q
- new net SRAM-11: MEM1001.A11, U1003.3Q
- new net SRAM-12: MEM1001.A12, U1003.4Q
- new net SRAM-13: MEM1001.A13, U1003.5Q
- new net SRAM-14: MEM1001.A14, U1003.6Q
- new net SRAM-15: MEM1001.A15, U1003.7Q
- new net SRAM-16: MEM1001.A16, U1001.GPIO-G14
- new net SRAM-17: MEM1001.A17, U1001.GPIO-G12
- new net SRAM-2: MEM1001.A2, U1002.2Q
- new net SRAM-3: MEM1001.A3, U1002.3Q
- new net SRAM-4: MEM1001.A4, U1002.4Q
- new net SRAM-5: MEM1001.A5, U1002.5Q
- new net SRAM-6: MEM1001.A6, U1002.6Q
- new net SRAM-7: MEM1001.A7, U1002.7Q
- new net SRAM-8: MEM1001.A8, U1003.0Q
- new net SRAM-9: MEM1001.A9, U1003.1Q
- new net SRST-MCLR: K1006.L1, R103.2, R104.1, TP2.TP
- new net STATUS: R101.1, U1001.GPIO-C12
- new net STATUS-LED: LED101.1, R101.2
- new net USB-PIN-1: U1001.V-USB-BUS, USB.P$1
- new net USB-PIN-2: U1001.USB-D-, USB.P$2
- new net USB-PIN-3: U1001.USB-D+, USB.P$3
- new net USB-V-TOGGLE: R907.1, U1001.GPIO-A10
- net 12V-INPUT: now also 12V.TP, R202.1; no longer 5V-REG.VIN, C1.1.1, C1.2.1, C22.1, D2.A, MAIN-SMPS.IN1, MAIN-SMPS.IN2, POWER.L, R10.1
- net 14V-RAIL: now also 14V.TP, DISP-1.4, DISP-2.4, DISP-3.4; no longer 14V-REG.OUT, C31.2, DISP-1.18, DISP-2.18, DISP-3.18, R32.2
- net 5V-RAIL: now also 5V.TP, AUX.P$1, K1001.L2, K1003.L2, R909.1, U1007.V+; no longer 5V-REG.VOUT, 5V-TOGGLE-1.L2, 5V-TOGGLE-2.L2, AUX-PRESS.P$1, C21.1, C8.1, EGT-AMP.VCC, R4.2, Y2.OE0, Y2.VCC
- net ACCEL-EN: now also R804.2, U1006.EN; no longer MMA8652FC.EN, R138.1
- net AN0-VOLT: now also F900.2, U1001.AN-0; no longer F0.1, PIC32MX.AN-0
- net AN1-BOOST: now also F901.2, U1001.AN-1; no longer F1.1, PIC32MX.AN-1
- net AN10: now also F910.1, P-10&11.2; no longer 10&11.2, F10.1
- net AN11: now also F911.1, P-10&11.3; no longer 10&11.3, F11.2
- net AN12: now also F912.1, P-12&13.2; no longer 12&13.2, F12.1
- net AN13: now also F913.1, P-12&13.3; no longer 12&13.3, F13.2
- net AN4: now also F904.2, P-4&5.2; no longer 4&5.2, F4.2
- net AN5: now also F905.2, P-4&5.3; no longer 4&5.3, F5.1
- net AN8: now also F908.1, P-8&9.2; no longer 8&9.2, F8.1
- net AN9: now also F909.1, P-8&9.3; no longer 8&9.3, F9.2
- net AUX-OUT: now also F903.1, R904.2, R905.1; no longer F2.2, R130.2, R131.1
- net BOOST-OUT: now also F901.1, U1005.V+; no longer F1.2, NBPLANN100PAUNV.V+
- net BOOST-PWR: now also K1001.L1, K1002.L2, U1005.VDD; no longer 3.3V-TOGGLE-2.L2, 5V-TOGGLE-2.L1, NBPLANN100PAUNV.VDD
- net BOOST-SSR: now also C901.2, K1001.C-, K1002.C+; no longer 3.3V-TOGGLE-2.C+, 5V-TOGGLE-2.C-, C11.2
- net DISP1-B1: now also DISP-1.11, U1001.SPI3-DI; no longer DISP-1.5, PIC32MX.SPI2-DI
- net DISP1-B2: now also DISP-1.12, U1008.D1; no longer DISP-1.11, PIC32MX.GPIO-E8
- net DISP1-B3: now also DISP-1.10, U1008.D0; no longer DISP-1.17, PIC32MX.GPIO-E9
- net DISP2-B1: now also DISP-2.11, U1001.SPI4-DI; no longer DISP-2.5, PIC32MX.SPI3-DI
- net DISP2-B2: now also DISP-2.12, U1008.D3; no longer DISP-2.11, PIC32MX.GPIO-C13
- net DISP2-B3: now also DISP-2.10, U1008.D2; no longer DISP-2.17, PIC32MX.GPIO-C14
- net DISP2-RS: now also DISP-2.5, U1001.SPI4-SS; no longer DISP-2.16, PIC32MX.GPIO-G14
- net DISP3-B1: now also DISP-3.11, U1001.SPI2-DI, U1008.Q7; no longer DISP-3.5, PIC32MX.SPI4-DI
- net DISP3-B2: now also DISP-3.12, U1008.D5; no longer DISP-3.11, PIC32MX.GPIO-G12
- net DISP3-B3: now also DISP-3.10, U1008.D4; no longer DISP-3.17, PIC32MX.GPIO-G13
- net DISP3-RS: now also DISP-3.5, U1001.SPI2-SS; no longer DISP-1.16, PIC32MX.GPIO-G15
- net EGT-NEG-IN: now also EGT.L, R901.2, R902.1, U1007.-IN; no longer EGT-AMP.IN-, EGT.R, R133.1, R136.1
- net EGT-OUT: now also F902.1, R902.2, U1007.OUT1; no longer EGT-AMP.OUT, F3.1, R133.2
- net EGT-POS-IN: now also EGT.R, U1007.+IN; no longer EGT-AMP.IN+, EGT.L
- net ICSP-SSR: now also C903.1, K1005.C-, K1006.C+; no longer 3.3V-TOGGLE-3.C+, 5V-TOGGLE-3.C-, C9.1
- net JTAG-PIN-1: now also TP1.TP, U1001.JTAG-MODE; no longer JTAG.1, PIC32MX.JTAG-MODE
- net JTAG-PIN-2: now also TP3.TP, U1001.JTAG-CLK-IN; no longer JTAG.2, PIC32MX.JTAG-CLK-IN
- net JTAG-PIN-3: now also TP4.TP, U1001.JTAG-DI; no longer JTAG.3, PIC32MX.JTAG-DI
- net JTAG-PIN-4: now also TP5.TP, U1001.JTAG-DO; no longer JTAG.4, PIC32MX.JTAG-DO
- net MCLR: now also R104.2, U1001.MCLR; no longer F14.1, PIC32MX.MCLR
- net MPL-BYP-CAP: now also C802.2, U1004.CAP; no longer C127.2, MPL3115A101.CAP
- net OIL-PRESS-OUT: now also AUX.P$3, R904.1; no longer AUX-PRESS.P$3, R131.2
- net PMA-LL: now also U1001.PMA-LL, U1002.LE; no longer LATCH-LOW.LE, PIC32MX.PMA-LL
- net PMD-14: now also MEM1001.I/O-14, R714.2, U1003.6D; no longer AS7C31026B.I/O-14, LATCH-HIGH.1D, PIC32MX.PMD-14
- net PMD0: now also R700.1, U1001.PMD-0; no longer AS7C31026B.I/O-0, LATCH-LOW.7D, PIC32MX.PMD-0
- net PMD1: now also R701.1, U1001.PMD-1; no longer AS7C31026B.I/O-1, LATCH-LOW.6D, PIC32MX.PMD-1
- net PMD10: now also R710.1, U1001.PMD-10; no longer AS7C31026B.I/O-10, LATCH-HIGH.5D, PIC32MX.PMD-10
- net PMD11: now also R711.1, U1001.PMD-11; no longer AS7C31026B.I/O-11, LATCH-HIGH.4D, PIC32MX.PMD-11
- net PMD12: now also R712.1, U1001.PMD-12; no longer AS7C31026B.I/O-12, LATCH-HIGH.3D, PIC32MX.PMD-12
- net PMD13: now also R713.1, U1001.PMD-13; no longer AS7C31026B.I/O-13, LATCH-HIGH.2D, PIC32MX.PMD-13
- net PMD15: now also R715.1, U1001.PMD-15; no longer AS7C31026B.I/O-15, LATCH-HIGH.0D, PIC32MX.PMD-15
- net PMD2: now also R702.1, U1001.PMD-2; no longer AS7C31026B.I/O-2, LATCH-LOW.5D, PIC32MX.PMD-2
- net PMD3: now also R703.1, U1001.PMD-3; no longer AS7C31026B.I/O-3, LATCH-LOW.4D, PIC32MX.PMD-3
- net PMD4: now also R704.1, U1001.PMD-4; no longer AS7C31026B.I/O-4, LATCH-LOW.3D, PIC32MX.PMD-4
- net PMD5: now also R705.1, U1001.PMD-5; no longer AS7C31026B.I/O-5, LATCH-LOW.2D, PIC32MX.PMD-5
- net PMD6: now also R706.1, U1001.PMD-6; no longer AS7C31026B.I/O-6, LATCH-LOW.1D, PIC32MX.PMD-6
- net PMD7: now also R707.1, U1001.PMD-7; no longer AS7C31026B.I/O-7, LATCH-LOW.0D, PIC32MX.PMD-7
- net PMD8: now also R708.1, U1001.PMD-8; no longer AS7C31026B.I/O-8, LATCH-HIGH.7D, PIC32MX.PMD-8
- net PMD9: now also R709.1, U1001.PMD-9; no longer AS7C31026B.I/O-9, LATCH-HIGH.6D, PIC32MX.PMD-9
- net PMP-CS1: now also MEM1001.CE, U1001.PMP-CS1, U1002.OE, U1003.OE; no longer LATCH-HIGH.OE, LATCH-LOW.OE, PIC32MX.PMP-CS1
- net PMP-WRITE: now also MEM1001.WE, U1001.PMP-ENB; no longer AS7C31026B.WE, PIC32MX.PMP-WR
- net SD-SPI-CLK: now also U1001.GPIO-G13, X3.P$3; no longer MICRO-SD.CLK, SC18IS602B.SPI-CLK
- net SPI2-CLK: now also DISP-2.15, U1001.SPI4-CLK; no longer DISP-1.3, PIC32MX.SPI2-CLK
- net SPI3-CLK: now also DISP-3.15, U1001.SPI2-CLK, U1008.CP; no longer DISP-2.3, PIC32MX.SPI3-CLK
- net USB-PWR: now also K1003.L1, K1004.L2, K1005.L2, P-10&11.1, P-12&13.1, P-4&5.1, P-8&9.1; no longer 10&11.1, 12&13.1, 3.3V-TOGGLE-1.L2, 4&5.1, 5V-TOGGLE-1.L1, 5V-TOGGLE-3.L2, 8&9.1
- net USB-SSR: now also C902.2, K1003.C-, K1004.C+; no longer 3.3V-TOGGLE-1.C+, 5V-TOGGLE-1.C-, C10.2
- net V-CAP: now also C102.1, U1001.V-CAP; no longer C124.2, PIC32MX.V-CAP
Other:
- note added: "(1)"
- note added: "(2)"
- note added: "(3)"
- note added: "(4)"
- note added: "**AN10 & AN11** Use uUSB-A Plug for ICSP"
- note added: "20 MHz, 2 ppm TCXO Oscillator"
- note added: "5V-3.3V Boost Resolution"
- note added: "5V-3.3V USB Autodetect"
- note added: "AN6&7-to-ICSP Swap Plug in uUSB-A Cable for ICSP Programming"
- note added: "Analog Inputs: 0-3.3V range Source: 5V @ 50 mA per pair"
- note added: "Analog, MCLR & HPD Supply"
- note added: "Digital & Osc Supply"
- note added: "Digital Input Control 1) I2C Pullups 2) Baro. & Thermo. 3) Accelerometer 4) Parallel-to-Serial Shift Register"
- note added: "Dispaly Outputs - Each port has 1xSPI, 3xButton, 2xPWM, 3.3V Rail, 14V Rail"
- note added: "Frame Buffer & General Buffer 4-Mbit SRAM, 120MHz 8 ns Propogation Delay"
- note added: "Ground Interconnects"
- note added: "ICSP Pins cannot have >100 ohms resistance 100 || 470 = ~82"
- note added: "Impulse Inputs RPM, VSS, etc."
- note added: "On-Board Analog Sensors 1) 100-psi-a 2) EGT 0-1100C 3) 5V Aux Input"
- note added: "Outside Communication 1) SD Card Conn. 2) CAN Bus Interface 3) FS USB Port 4) JTAG Header"
- note added: "PIC32MX795-Driven Digital Gauge & DAQ x14 Analog Input, x3 Impulse Input x3 Display Output, 4-Mbit SRAM SD Card Storage, USB Device, CAN Bus ICSP & JTAG Prog. and Diag. Support"
- note added: "Power Supply Taps"
- note added: "SRAM & Imp. Supply"
- note added: "Schematic Capture for D-DAQ Version: Proto v4 Released Under CERN OHL v1.2"
- note added: "Solid State Relays - SSRs 1) Change Press. Sensor Res. 2) Autodetect for AN Sensors"
- note added: "Termination of Parallel lines"
- note removed: "Schematic Capture for D-DAQ Version: Proto v3.6.5 Released Under CERN OHL v1.2"
- moved on the sheet: DISP-1, DISP-2, DISP-3
